File: hardware/FlockOff/FlockOff.kicad_pcb (KiCad board)
At the start: 2 copper layers, 73.5 x 34.5 mm, 5 parts, among them U1 XIAO-ESP32-S3-DIP

Commit message: moar logging
Routing:
- net GND: track 3.37 -> 1.04 mm
- net Net-(D1-Vcc): track 20.2 -> 20.8 mm
Changed lines of the file:
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@@
 			)
 		)
-		(pad "1" thru_hole circle
+		(pad "1" thru_hole oval
 			(at 1.95 0)
-			(size 1.1 1.1)
+			(size 1.1 2.2)
 			(drill 0.8)
 			(layers "*.Cu" "*.Mask")
@@
 			(pintype "input")
 		)
-		(pad "2" thru_hole circle
+		(pad "2" thru_hole oval
 			(at 0.65 0)
-			(size 1.1 1.1)
+			(size 1.1 2.2)
 			(drill 0.8)
 			(layers "*.Cu" "*.Mask")
@@
 			(pintype "power_in")
 		)
-		(pad "3" thru_hole circle
+		(pad "3" thru_hole oval
 			(at -0.65 0)
-			(size 1.1 1.1)
+			(size 1.1 2.2)
 			(drill 0.8)
 			(layers "*.Cu" "*.Mask")
@@
 			(pintype "power_in")
 		)
-		(pad "4" thru_hole circle
+		(pad "4" thru_hole oval
 			(at -1.95 0)
-			(size 1.1 1.1)
+			(size 1.1 2.2)
 			(drill 0.8)
 			(layers "*.Cu" "*.Mask")
@@
 			)
 		)
-		(pad "1" thru_hole circle
+		(pad "1" thru_hole oval
 			(at 1.95 0 180)
-			(size 1.1 1.1)
+			(size 1.1 2.2)
 			(drill 0.8)
 			(layers "*.Cu" "*.Mask")
@@
 			(pintype "input")
 		)
-		(pad "2" thru_hole circle
+		(pad "2" thru_hole oval
 			(at 0.65 0 180)
-			(size 1.1 1.1)
+			(size 1.1 2.2)
 			(drill 0.8)
 			(layers "*.Cu" "*.Mask")
@@
 			(pintype "power_in")
 		)
-		(pad "3" thru_hole circle
+		(pad "3" thru_hole oval
 			(at -0.65 0 180)
-			(size 1.1 1.1)
+			(size 1.2 2.2)
 			(drill 0.8)
 			(layers "*.Cu" "*.Mask")
@@
 			(pintype "power_in")
 		)
-		(pad "4" thru_hole circle
+		(pad "4" thru_hole oval
 			(at -1.95 0 180)
-			(size 1.1 1.1)
+			(size 1.1 2.2)
 			(drill 0.8)
 			(layers "*.Cu" "*.Mask")
@@
 	)
 	(segment
-		(start 171.3 86)
-		(end 171.3 84.8)
+		(start 169.5 100.4)
+		(end 169.6 100.5)
 		(width 0.2)
 		(layer "B.Cu")
@@
 	)
 	(segment
-		(start 169.6 100.5)
-		(end 170.1 101)
+		(start 169.5 99.5)
+		(end 169.5 100.4)
 		(width 0.2)
 		(layer "B.Cu")
@@
 	)
 	(segment
-		(start 169.5 100.4)
-		(end 169.6 100.5)
-		(width 0.2)
-		(layer "B.Cu")
-		(net 1)
-	)
-	(segment
-		(start 169.5 99.5)
-		(end 169.5 100.4)
-		(width 0.2)
-		(layer "B.Cu")
-		(net 1)
-	)
-	(segment
-		(start 171.3 84.8)
-		(end 171.6 84.5)
-		(width 0.2)
-		(layer "B.Cu")
-		(net 1)
-	)
-	(segment
 		(start 146 85.835)
 		(end 146 85.5)
@@
 	)
 	(segment
-		(start 166.81 89.19)
-		(end 170 86)
-		(width 0.2)
-		(layer "F.Cu")
-		(net 3)
-	)
-	(segment
 		(start 163.1 89.19)
 		(end 166.81 89.19)
@@
 	)
 	(segment
-		(start 172.1 86.5)
+		(start 166.81 89.19)
+		(end 167.81 89.19)
+		(width 0.2)
+		(layer "F.Cu")
+		(net 3)
+	)
+	(segment
+		(start 167.81 89.19)
+		(end 170 87)
+		(width 0.2)
+		(layer "F.Cu")
+		(net 3)
+	)
+	(segment
+		(start 170 87)
+		(end 170 86)
+		(width 0.2)
+		(layer "F.Cu")
+		(net 3)
+	)
+	(segment
+		(start 172.1 99.5)
+		(end 172.5 99.1)
+		(width 0.2)
+		(layer "F.Cu")
+		(net 4)
+	)
+	(segment
+		(start 172.5 86.1)
 		(end 172.6 86)
 		(width 0.2)
@@
 	)
 	(segment
-		(start 172.1 99.5)
-		(end 172.1 86.5)
-		(width 0.2)
-		(layer "F.Cu")
+		(start 172.5 99.1)
+		(end 172.5 86.1)
+		(width 0.2)
+		(layer "F.Cu")
